File: schematics/UE1-TTL-Clock/bell.kicad_sch (KiCad schematic)
At the start: 7 parts, among them U4 NE555

Commit message: Lay out clock board
Other:
- title: UE1- TTL Clock and Diagnostics -> UE1-TTL Clock and Front Panel
Changed lines of the file:
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@@
 	(paper "A4")
 	(title_block
-		(title "UE1- TTL Clock and Diagnostics")
+		(title "UE1-TTL Clock and Front Panel")
 		(date "2025")
 		(rev "1")
