File: schematics/UE1-TTL-Memory/input_register.kicad_sch (KiCad schematic)
At the start: 11 parts, among them SW1 Inputs, U4 74LS125, U5 74LS151

Commit message: Lay out memory board
Parts:
- removed U4: 74LS125, Package_DIP:DIP-14_W7.62mm, symbol 74xx:74LS125
- removed U5: 74LS151, Package_DIP:DIP-16_W7.62mm, symbol 74xx:74LS151
- added U4: 74LS251, Package_DIP:DIP-16_W7.62mm, symbol 74xx:74LS251
- SW1: footprint Button_Switch_THT:SW_DIP_SPSTx08_Slide_9.78x22.5mm_W7.62mm_P2.54mm -> Button_Switch_THT:SW_DIP_SPSTx08_Slide_6.7x21.88mm_W7.62mm_P2.54mm_LowProfile
- renumbered C5 to C4
Connections:
- net +5V: now also SW1.16, U4.16 (VCC); no longer SW1.9
- net GND: now also U4.8 (GND)
- net IR1: now also SW1.7, U4.3 (I1); no longer SW1.8
- net IR2: now also SW1.6, U4.2 (I2); no longer SW1.7
- net IR3: now also SW1.5, U4.1 (I3); no longer SW1.6
- net IR4: now also SW1.4, U4.15 (I4); no longer SW1.5
- net IR5: now also SW1.3, U4.14 (I5); no longer SW1.4
- net IR6: now also SW1.2, U4.13 (I6); no longer SW1.3
- net IR7: now also SW1.1, U4.12 (I7); no longer SW1.2
- net MEM0: now also U4.11 (S0)
- net MEM1: now also U4.10 (S1)
- net MEM2: now also U4.9 (S2)
- net RD_DATA: now also U4.5 (Y)
- net RR: now also U4.4 (I0)
- net ~{RD_IR}: now also U4.7 (~{OE})
Other:
- moved on the sheet: SW1
