File: schematics/UE1-TTL-Memory/output_register.kicad_sch (KiCad schematic)
At the start: 18 parts, among them U6 74LS259

Commit message: Lay out memory board
Parts:
- renumbered C6 to C5, U6 to U5
Other:
- note added: "Choose RLED values to match the properties of the LED's you are using. RLED = (5 - VLED) / ILED Examples: VLED = 1.7V, ILED = 15mA, RLED = 220R VLED = 1.9V, ILED = 2mA, RLED = 1550R (1K8 should be fine) VLED = 1.9V, ILED = 10mA, RLED = 310R (330R should be fine) Recommend 2mA LED's to reduce current draw on TTL outputs"
- note removed: "470R for 5mA rated LED's, 220R for 15mA rated LED's"
Changed lines of the file:
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@@
 		)
 	)
-	(text "470R for 5mA rated LED's, 220R for 15mA rated LED's"
-		(exclude_from_sim no)
-		(at 123.952 125.984 0)
+	(text "Choose RLED values to match the properties of the LED's you are using.\n\n        RLED = (5 - VLED) / ILED\n\nExamples:\n\n        VLED = 1.7V, ILED = 15mA, RLED = 220R\n        VLED = 1.9V, ILED =  2mA, RLED = 1550R (1K8 should be fine)\n        VLED = 1.9V, ILED = 10mA, RLED = 310R (330R should be fine)\n\nRecommend 2mA LED's to reduce current draw on TTL outputs"
+		(exclude_from_sim no)
+		(at 46.228 163.83 0)
 		(effects
 			(font
@@
 		(dnp no)
 		(fields_autoplaced yes)
-		(property "Reference" "#PWR44"
+		(property "Reference" "#PWR34"
 			(at 110.49 121.92 0)
 			(effects
@@
 			(project "UE1-Memory"
 				(path "/3387ba40-0694-43b2-a156-d12ce9552f1f/4783696b-edb1-49fa-83d3-8dbb9585c153"
-					(reference "#PWR44")
+					(reference "#PWR34")
 					(unit 1)
 				)
@@
 		(dnp no)
 		(fields_autoplaced yes)
-		(property "Reference" "#PWR41"
+		(property "Reference" "#PWR31"
 			(at 87.63 107.95 0)
 			(effects
@@
 			(project "UE1-Memory"
 				(path "/3387ba40-0694-43b2-a156-d12ce9552f1f/4783696b-edb1-49fa-83d3-8dbb9585c153"
-					(reference "#PWR41")
+					(reference "#PWR31")
 					(unit 1)
 				)
@@
 		(dnp no)
 		(fields_autoplaced yes)
-		(property "Reference" "#PWR47"
+		(property "Reference" "#PWR37"
 			(at 144.78 121.92 0)
 			(effects
@@
 			(project "UE1-Memory"
 				(path "/3387ba40-0694-43b2-a156-d12ce9552f1f/4783696b-edb1-49fa-83d3-8dbb9585c153"
-					(reference "#PWR47")
+					(reference "#PWR37")
 					(unit 1)
 				)
@@
 		(dnp no)
 		(fields_autoplaced yes)
-		(property "Reference" "#PWR42"
+		(property "Reference" "#PWR32"
 			(at 87.63 125.73 0)
 			(effects
@@
 			(project "UE1-Memory"
 				(path "/3387ba40-0694-43b2-a156-d12ce9552f1f/4783696b-edb1-49fa-83d3-8dbb9585c153"
-					(reference "#PWR42")
+					(reference "#PWR32")
 					(unit 1)
 				)
@@
 		(dnp no)
 		(fields_autoplaced yes)
-		(property "Reference" "#PWR51"
+		(property "Reference" "#PWR41"
 			(at 190.5 121.92 0)
 			(effects
@@
 			(project "UE1-Memory"
 				(path "/3387ba40-0694-43b2-a156-d12ce9552f1f/4783696b-edb1-49fa-83d3-8dbb9585c153"
-					(reference "#PWR51")
+					(reference "#PWR41")
 					(unit 1)
 				)
@@
 		(dnp no)
 		(fields_autoplaced yes)
-		(property "Reference" "#PWR40"
+		(property "Reference" "#PWR30"
 			(at 87.63 69.85 0)
 			(effects
@@
 			(project "UE1-Memory"
 				(path "/3387ba40-0694-43b2-a156-d12ce9552f1f/4783696b-edb1-49fa-83d3-8dbb9585c153"
-					(reference "#PWR40")
+					(reference "#PWR30")
 					(unit 1)
 				)
@@
 		(dnp no)
 		(fields_autoplaced yes)
-		(property "Reference" "#PWR48"
+		(property "Reference" "#PWR38"
 			(at 156.21 121.92 0)
 			(effects
@@
 			(project "UE1-Memory"
 				(path "/3387ba40-0694-43b2-a156-d12ce9552f1f/4783696b-edb1-49fa-83d3-8dbb9585c153"
-					(reference "#PWR48")
+					(reference "#PWR38")
 					(unit 1)
 				)
@@
 		(dnp no)
 		(fields_autoplaced yes)
-		(property "Reference" "#PWR49"
+		(property "Reference" "#PWR39"
 			(at 167.64 121.92 0)
 			(effects
@@
 			(project "UE1-Memory"
 				(path "/3387ba40-0694-43b2-a156-d12ce9552f1f/4783696b-edb1-49fa-83d3-8dbb9585c153"
-					(reference "#PWR49")
+					(reference "#PWR39")
 					(unit 1)
 				)
@@
 		(dnp no)
 		(fields_autoplaced yes)
-		(property "Reference" "#PWR43"
+		(property "Reference" "#PWR33"
 			(at 87.63 135.89 0)
 			(effects
@@
 			(project "UE1-Memory"
 				(path "/3387ba40-0694-43b2-a156-d12ce9552f1f/4783696b-edb1-49fa-83d3-8dbb9585c153"
-					(reference "#PWR43")
+					(reference "#PWR33")
 					(unit 1)
 				)
@@
 		(dnp no)
 		(fields_autoplaced yes)
-		(property "Reference" "C6"
+		(property "Reference" "C5"
 			(at 91.44 124.4599 0)
 			(effects
@@
 			(project "UE1-Memory"
 				(path "/3387ba40-0694-43b2-a156-d12ce9552f1f/4783696b-edb1-49fa-83d3-8dbb9585c153"
-					(reference "C6")
+					(reference "C5")
 					(unit 1)
 				)
@@
 		(dnp no)
 		(fields_autoplaced yes)
-		(property "Reference" "U6"
+		(property "Reference" "U5"
 			(at 89.8241 66.04 0)
 			(effects
@@
 			(project "UE1-Memory"
 				(path "/3387ba40-0694-43b2-a156-d12ce9552f1f/4783696b-edb1-49fa-83d3-8dbb9585c153"
-					(reference "U6")
+					(reference "U5")
 					(unit 1)
 				)
@@
 		(dnp no)
 		(fields_autoplaced yes)
-		(property "Reference" "#PWR50"
+		(property "Reference" "#PWR40"
 			(at 179.07 121.92 0)
 			(effects
@@
 			(project "UE1-Memory"
 				(path "/3387ba40-0694-43b2-a156-d12ce9552f1f/4783696b-edb1-49fa-83d3-8dbb9585c153"
-					(reference "#PWR50")
+					(reference "#PWR40")
 					(unit 1)
 				)
@@
 		(dnp no)
 		(fields_autoplaced yes)
-		(property "Reference" "#PWR46"
+		(property "Reference" "#PWR36"
 			(at 133.35 121.92 0)
 			(effects
@@
 			(project "UE1-Memory"
 				(path "/3387ba40-0694-43b2-a156-d12ce9552f1f/4783696b-edb1-49fa-83d3-8dbb9585c153"
-					(reference "#PWR46")
+					(reference "#PWR36")
 					(unit 1)
 				)
@@
 		(dnp no)
 		(fields_autoplaced yes)
-		(property "Reference" "#PWR45"
+		(property "Reference" "#PWR35"
 			(at 121.92 121.92 0)
 			(effects
@@
 			(project "UE1-Memory"
 				(path "/3387ba40-0694-43b2-a156-d12ce9552f1f/4783696b-edb1-49fa-83d3-8dbb9585c153"
-					(reference "#PWR45")
-					(unit 1)
-				)
+					(reference "#PWR35")
+					(unit 1)
+				)
